File: LEDmodule/communication.kicad_sch (KiCad schematic)
At the start: 0 parts

Commit message: Add start of comm's
Parts:
- added C3: 100n, symbol Device:C
- added C4, C5: C, symbol Device:C
- added D5: SM24-02HTG, Package_TO_SOT_SMD:SOT-323_SC-70, symbol Power_Protection:SP0502BAJT
- added D6: SMAJ24CA, Diode_SMD:D_SMA, symbol Diode:SMAJ24CA
- added R2: R, symbol Device:R
- added R3, R4: 10, symbol Device:R
- added U2: THVD8010, Package_TO_SOT_SMD:SOT-23-8, symbol Interface_UART:THVD8000
Connections:
- net +5V: now also C3.1, U2.8 (VCC)
- net Data1: now also C5.2
- net Data2: now also C4.2
- net GND: now also C3.2, D5.3 (A), R2.1, U2.5 (GND)
- new net: R2.2, U2.3 (F_SET)
- new net: R3.1, U2.6 (A)
- new net: R4.1, U2.7 (B)
- new net: C5.1, D5.1 (K), D6.2 (A2), R3.2
- new net: C4.1, D5.2 (K), D6.1 (A1), R4.2
- new net RS485.D: U2.4 (D)
- new net RS485.MODE: U2.2 (MODE)
- new net RS485.R: U2.1 (R)
Other:
- note added: "pulse proof"
