File: LEDmodule/mcu.kicad_sch (KiCad schematic)
At the start: 0 parts

Commit message: Finalize Led&Driver
Changed lines of the file:
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@@
+		)
+	)
+	(hierarchical_label "LP5015_EN"
+		(shape output)
+		(at 147.32 113.03 180)
+		(effects
+			(font
+				(size 1.27 1.27)
+			)
+			(justify right)
 		)
 	)
@@
 		(dnp no)
 		(fields_autoplaced yes)
-		(property "Reference" "#PWR07"
+		(property "Reference" "#PWR7"
 			(at 146.05 86.36 0)
 			(effects
@@
 			(project "LEDmodule"
 				(path "/80a08b48-2579-42cd-b65f-533f20aa7c1b/ae29019f-e893-4856-ad54-7d13fdb497b0"
-					(reference "#PWR07")
+					(reference "#PWR7")
 					(unit 1)
 				)
@@
 		(dnp no)
 		(fields_autoplaced yes)
-		(property "Reference" "#PWR08"
+		(property "Reference" "#PWR8"
 			(at 170.18 53.34 0)
 			(effects
@@
 			(project "LEDmodule"
 				(path "/80a08b48-2579-42cd-b65f-533f20aa7c1b/ae29019f-e893-4856-ad54-7d13fdb497b0"
-					(reference "#PWR08")
+					(reference "#PWR8")
 					(unit 1)
 				)

Commit message: Add start of comm's
Changed lines of the file:
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@@
 	)
 	(bus_entry
-		(at 170.18 83.82)
+		(at 196.85 91.44)
 		(size -2.54 2.54)
 		(stroke
@@
 	)
 	(bus_entry
-		(at 119.38 59.69)
+		(at 99.06 85.09)
 		(size 2.54 -2.54)
 		(stroke
@@
 	)
 	(bus_entry
-		(at 119.38 57.15)
+		(at 99.06 82.55)
 		(size 2.54 -2.54)
 		(stroke
@@
 	)
 	(bus_entry
-		(at 170.18 80.01)
+		(at 196.85 87.63)
 		(size -2.54 2.54)
 		(stroke
@@
 	)
 	(bus_entry
-		(at 119.38 62.23)
+		(at 99.06 87.63)
 		(size 2.54 -2.54)
 		(stroke
@@
 	(bus
 		(pts
-			(xy 170.18 76.2) (xy 195.58 76.2)
-		)
-		(stroke
-			(width 0)
-			(type default)
-		)
-	)
-	(bus
-		(pts
-			(xy 170.18 76.2) (xy 170.18 80.01)
-		)
-		(stroke
-			(width 0)
-			(type default)
-		)
-	)
-	(bus
-		(pts
-			(xy 121.92 57.15) (xy 121.92 54.61)
-		)
-		(stroke
-			(width 0)
-			(type default)
-		)
-	)
-	(wire
-		(pts
-			(xy 165.1 82.55) (xy 167.64 82.55)
-		)
-		(stroke
-			(width 0)
-			(type default)
-		)
-	)
-	(wire
-		(pts
-			(xy 116.84 62.23) (xy 119.38 62.23)
-		)
-		(stroke
-			(width 0)
-			(type default)
-		)
-	)
-	(wire
-		(pts
-			(xy 165.1 86.36) (xy 167.64 86.36)
-		)
-		(stroke
-			(width 0)
-			(type default)
-		)
-	)
-	(wire
-		(pts
-			(xy 116.84 59.69) (xy 119.38 59.69)
-		)
-		(stroke
-			(width 0)
-			(type default)
-		)
-	)
-	(wire
-		(pts
-			(xy 116.84 57.15) (xy 119.38 57.15)
-		)
-		(stroke
-			(width 0)
-			(type default)
-		)
-	)
-	(bus
-		(pts
-			(xy 121.92 59.69) (xy 121.92 57.15)
-		)
-		(stroke
-			(width 0)
-			(type default)
-		)
-	)
-	(bus
-		(pts
-			(xy 170.18 80.01) (xy 170.18 83.82)
-		)
-		(stroke
-			(width 0)
-			(type default)
-		)
-	)
-	(bus
-		(pts
-			(xy 121.92 54.61) (xy 121.92 52.07)
-		)
-		(stroke
-			(width 0)
-			(type default)
-		)
-	)
-	(bus
-		(pts
-			(xy 121.92 52.07) (xy 133.35 52.07)
+			(xy 196.85 83.82) (xy 222.25 83.82)
+		)
+		(stroke
+			(width 0)
+			(type default)
+		)
+	)
+	(bus
+		(pts
+			(xy 196.85 83.82) (xy 196.85 87.63)
+		)
+		(stroke
+			(width 0)
+			(type default)
+		)
+	)
+	(bus
+		(pts
+			(xy 101.6 82.55) (xy 101.6 80.01)
+		)
+		(stroke
+			(width 0)
+			(type default)
+		)
+	)
+	(wire
+		(pts
+			(xy 191.77 90.17) (xy 194.31 90.17)
+		)
+		(stroke
+			(width 0)
+			(type default)
+		)
+	)
+	(wire
+		(pts
+			(xy 96.52 87.63) (xy 99.06 87.63)
+		)
+		(stroke
+			(width 0)
+			(type default)
+		)
+	)
+	(wire
+		(pts
+			(xy 191.77 93.98) (xy 194.31 93.98)
+		)
+		(stroke
+			(width 0)
+			(type default)
+		)
+	)
+	(wire
+		(pts
+			(xy 96.52 85.09) (xy 99.06 85.09)
+		)
+		(stroke
+			(width 0)
+			(type default)
+		)
+	)
+	(wire
+		(pts
+			(xy 96.52 82.55) (xy 99.06 82.55)
+		)
+		(stroke
+			(width 0)
+			(type default)
+		)
+	)
+	(bus
+		(pts
+			(xy 101.6 85.09) (xy 101.6 82.55)
+		)
+		(stroke
+			(width 0)
+			(type default)
+		)
+	)
+	(bus
+		(pts
+			(xy 196.85 87.63) (xy 196.85 91.44)
+		)
+		(stroke
+			(width 0)
+			(type default)
+		)
+	)
+	(bus
+		(pts
+			(xy 101.6 80.01) (xy 101.6 77.47)
+		)
+		(stroke
+			(width 0)
+			(type default)
+		)
+	)
+	(bus
+		(pts
+			(xy 101.6 77.47) (xy 113.03 77.47)
 		)
 		(stroke
@@
 	)
 	(label "MODE"
-		(at 116.84 62.23 180)
+		(at 96.52 87.63 180)
 		(effects
 			(font
@@
 	)
 	(label "RS485{R D MODE}"
-		(at 127 52.07 180)
+		(at 106.68 77.47 180)
 		(effects
 			(font
@@
 	)
 	(label "R"
-		(at 116.84 57.15 180)
+		(at 96.52 82.55 180)
 		(effects
 			(font
@@
 	)
 	(label "SDA"
-		(at 165.1 86.36 180)
+		(at 191.77 93.98 180)
 		(effects
 			(font
@@
 	)
 	(label "I2C{SCL SDA}"
-		(at 185.42 76.2 180)
+		(at 212.09 83.82 180)
 		(effects
 			(font
@@
 	)
 	(label "SCL"
-		(at 165.1 82.55 180)
+		(at 191.77 90.17 180)
 		(effects
 			(font
@@
 	)
 	(label "D"
-		(at 116.84 59.69 180)
+		(at 96.52 85.09 180)
 		(effects
 			(font
@@
 	(hierarchical_label "comm"
 		(shape bidirectional)
-		(at 133.35 52.07 0)
+		(at 113.03 77.47 0)
 		(effects
 			(font
@@
 	(hierarchical_label "I2C"
 		(shape bidirectional)
-		(at 195.58 76.2 0)
+		(at 222.25 83.82 0)
 		(effects
 			(font
@@
 	(hierarchical_label "LP5015_EN"
 		(shape output)
-		(at 147.32 113.03 180)
-		(effects
-			(font
-				(size 1.27 1.27)
-			)
-			(justify right)
+		(at 196.85 77.47 0)
+		(effects
+			(font
+				(size 1.27 1.27)
+			)
+			(justify left)
 		)
 	)
 	(symbol
 		(lib_id "power:GND")
-		(at 146.05 80.01 0)
+		(at 173.99 102.87 0)
 		(unit 1)
 		(exclude_from_sim no)
@@
 		(fields_autoplaced yes)
 		(property "Reference" "#PWR7"
-			(at 146.05 86.36 0)
+			(at 173.99 109.22 0)
 			(effects
 				(font
@@
 		)
 		(property "Value" "GND"
-			(at 146.05 85.09 0)
+			(at 173.99 107.95 0)
 			(effects
 				(font
@@
 		)
 		(property "Footprint" ""
-			(at 146.05 80.01 0)
+			(at 173.99 102.87 0)
 			(effects
 				(font
@@
 		)
 		(property "Datasheet" ""
-			(at 146.05 80.01 0)
+			(at 173.99 102.87 0)
 			(effects
 				(font
@@
 		)
 		(property "Description" "Power symbol creates a global label with name \"GND\" , ground"
-			(at 146.05 80.01 0)
+			(at 173.99 102.87 0)
 			(effects
 				(font
@@
 	(symbol
 		(lib_id "power:+5V")
-		(at 170.18 49.53 0)
+		(at 172.72 58.42 0)
 		(unit 1)
 		(exclude_from_sim no)
@@
 		(fields_autoplaced yes)
 		(property "Reference" "#PWR8"
-			(at 170.18 53.34 0)
+			(at 172.72 62.23 0)
 			(effects
 				(font
@@
 		)
 		(property "Value" "+5V"
-			(at 170.18 44.45 0)
+			(at 172.72 53.34 0)
 			(effects
 				(font
@@
 		)
 		(property "Footprint" ""
-			(at 170.18 49.53 0)
+			(at 172.72 58.42 0)
 			(effects
 				(font
@@
 		)
 		(property "Datasheet" ""
-			(at 170.18 49.53 0)
+			(at 172.72 58.42 0)
 			(effects
 				(font
@@
 		)
 		(property "Description" "Power symbol creates a global label with name \"+5V\""
-			(at 170.18 49.53 0)
-			(effects
-				(font
+			(at 172.72 58.42 0)
+			(effects
+				(font
